File: Documents/Eagle/ardBeeQueen.sch (EAGLE design)
At the start: 12 parts

Commit message: updated eagle docs
Changed lines of the file:
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@@
 <pinref part="U$1" gate="G$1" pin="D3"/>
 <pinref part="SV2" gate="G$1" pin="SIG"/>
-<wire x1="152.4" y1="190.5" x2="223.52" y2="190.5" width="0.1524" layer="91"/>
+<wire x1="223.52" y1="190.5" x2="152.4" y2="190.5" width="0.1524" layer="91"/>
 </segment>
 </net>
 <net name="N$14" class="0">
 <segment>
-<wire x1="170.18" y1="172.72" x2="170.18" y2="187.96" width="0.1524" layer="91"/>
 <wire x1="170.18" y1="187.96" x2="223.52" y2="187.96" width="0.1524" layer="91"/>
 <pinref part="U$1" gate="G$1" pin="D4"/>
+<wire x1="170.18" y1="187.96" x2="170.18" y2="172.72" width="0.1524" layer="91"/>
 <pinref part="SV3" gate="G$1" pin="SIG"/>
-<wire x1="152.4" y1="172.72" x2="170.18" y2="172.72" width="0.1524" layer="91"/>
+<wire x1="170.18" y1="172.72" x2="152.4" y2="172.72" width="0.1524" layer="91"/>
 </segment>
 </net>
