File: Documents/Eagle/ardBeeQueenWMountHoles50x52.brd (EAGLE design)
At the start: 54.8 x 57.1 mm, 12 parts

Commit message: upd
Parts:
- moved SV5 22.9 mm to (36.8, 55.9)
- moved J1 6.35 mm to (33.0, 93.3)
- moved SV1 6.35 mm to (8.89, 54.6)
- moved SV2 6.35 mm to (12.7, 93.3)
- moved SV3 6.35 mm to (21.6, 93.3)
- moved SV4 6.35 mm to (32.4, 55.9)
Routing:
- net N$1: track 65.0 -> 57.8 mm
- net N$7: track 22.6 -> 21.3 mm
- net N$4: track 21.5 -> 22.8 mm
- net N$8: track 28.7 -> 27.4 mm
- net N$2: track 30.5 -> 31.9 mm
- net N$3: track 18.4 -> 19.4 mm
- net N$16: track 119.9 -> 120.6 mm
- net N$6: track 11.1 -> 10.5 mm
- net N$5: track 7.36 -> 6.86 mm
