File: Documents/Eagle/ardBeeQueen_12-pin_lcd.sch (EAGLE design)
At the start: 12 parts

Commit message: Eagle update
Parts:
- added SV5: (no value), myLib-01-Headers:POWER_IN-2-PIN_FEMALE_HEADER
- J1: device myLib-01-Headers:DHT22_4-PIN_FEMALE_HEADERPTH -> myLib-01-Headers:DHT22_3-PIN_FEMALE_HEADER
- R1: value 10K -> 10k; device pot:TRIM_EU-B25P -> myLib-04-OftenUsed:POTENTIOMETER_CA6VCA6V
Connections:
- removed net N$16: C1.2, C2.2, J1.GND, R1.A, SV1.GND, SV2.GND, SV3.GND, SV4.GND, SV6.GND, SV6.LED-, SV6.R/W, U$1.GND
- new net GND: C1.2, C2.2, J1.GND, R1.A, SV1.GND, SV2.GND, SV3.GND, SV4.GND, SV5.GND, SV6.GND, SV6.LED-, SV6.R/W, U$1.GND
- net N$17: now also SV5.VCC
Other:
- note added: "5V Input"
- note added: "DHT Temperature Sensor"
- note added: "Fan Relay"
- note added: "Heater Relay"
- note added: "LCD"
- note added: "Rotary Encoder"
